File: pinned/core/kicad/core.kicad_pcb (KiCad board)
At the start: 4 copper layers, 120 x 100 mm, 282 parts, among them J1 USB4105-GF-A-120, J10 SPK B L, J11 SPK B R, J2 HR911105A, J3 FFC 20P, J4 SUB OUT, J5 LINE IN, J6 SPK A L, J7 SPK A R, Q1 AO4485, Q2 2N7002, Q3 S8050, Q4 S8050, Q5 S8050, Q6 S8050, SW1 EC11, SW2 BTN1, SW3 BTN2, U1 CH224Q, U10 ES9018K2M, U11 OPA1678, U12 PCM5102A, U13 ES7243E, U14 TS5A23157, U15 TPA3221, U16 TPA3221, U17 TCA9555, U18 IRM-H638T, U19 PLR237/T8BK, U2 USBLC6-2SC6, U3 INA186A1, U4 SY8303AIC, U5 SY8089A1AAC, U6 LP5907-3.3, U7 ESP32-WROVER-E-N8R8, U8 CH340C, U9 LAN8720A, Y1 50MHz, Y2 50MHz

Commit message: hwde's score reads the hi-fi boards as they are now: re-pin core and lite-main at hifi-receiver-2 main, add ultra-front
* hwde's score reads the hi-fi boards as they are now: core and lite-ma…

…in re-pinned at hifi-receiver-2 56e91aa, ultra-front added

The re-pin is a new baseline (docs/score.md): 9da177ca's review-2 ECO scripts are
classified as stand-ins with the gap each fills.

* merge main
Parts:
- added C130: 470pF, aiee:C0603, F.Cu at (96.5, 144.0)
- added C131: 1uF, aiee:C0402, F.Cu at (99.3, 140.8)
- added C132: 100nF, aiee:C0402, F.Cu at (100.9, 157.7)
- added C136: 470pF, aiee:C0603, F.Cu at (102.1, 144.0)
- added C137: 1uF, aiee:C0402, F.Cu at (99.3, 144.0)
- added Q7: S8050, aiee:SOT-23-3_L3.0-W1.7-P0.95-LS2.9-BR, F.Cu at (103.7, 149.0)
- added R130: 150k, aiee:R0603, F.Cu at (96.5, 140.8)
- added R131: 10k, aiee:R0402, F.Cu at (96.5, 142.4)
- added R132: 100k, aiee:R0402, F.Cu at (99.3, 142.4)
- added R133: 47k, aiee:R0402, F.Cu at (106.6, 155.0)
- added R134: 100k, aiee:R0402, F.Cu at (106.8, 157.0)
- added R135: 10k, aiee:R0402, F.Cu at (101.5, 159.2)
- added R136: 150k, aiee:R0603, F.Cu at (102.1, 140.8)
- added R137: 10k, aiee:R0402, F.Cu at (102.1, 142.4)
- added R138: 100k, aiee:R0402, F.Cu at (99.3, 145.4)
- added R149: 100k, aiee:R0402, F.Cu at (94.2, 145.1)
- added R150: 100k, aiee:R0402, F.Cu at (102.8, 145.7)
- added R20: 10k, aiee:R0402, F.Cu at (52.2, 185.5)
- added U20: TS5A23157, aiee:MSOP-10_L3.0-W3.0-P0.50-LS5.0-BL, F.Cu at (103.8, 154.2)
- C101, C102, C111, C112: value 1uF -> 4.7uF; footprint aiee:C0402 -> aiee:C0603
- C47: value 100nF -> 1uF
- C8: value 1uF -> 2.2uF
- J1: value USB4105-GF-A-120 -> USB4085-GF-A; footprint aiee:USB-C-SMD_MC-311D -> aiee:USC-C-SMD_USB4085-GF-A
- R4, R5: value 100k -> 470k
- R45: value 100k -> 2.2k
- R73, R75, R81, R83: value 1.5k -> 1.3k
- U17: value TCA9555 -> TCA9539
- U18: value IRM-H638T -> IRM-3638T; footprint aiee:SENSOR-SMD_IRM-H638T-TR2-TL -> aiee:OPTO-TH_IRM-3638T
- U8: value CH340C -> CH340B
- Y1: value 50MHz -> 49.152MHz
- moved C111 11.8 mm to (131.3, 159.0), turned to 90 degrees
- moved C101 11.4 mm to (131.3, 156.0)
- moved C112 9.46 mm to (140.3, 153.5)
- moved C102 0.42 mm to (138.3, 149.2), turned to 0 degrees
- moved J1 0.08 mm to (38.5, 178.7)
Connections:
- net /amp_a/A_SPK_L+ renamed /A_SPK_L+
- net /amp_a/A_SPK_R+ renamed /A_SPK_R+
- C101 pad 1: /linein/LDIV_L -> /linein/ADC_SRC_L
- C111 pad 1: /linein/LDIV_R -> /linein/ADC_SRC_R
- Q2 pad 2: GND -> /power_in/PD_PG
- R57 pad 1: +3V3 -> /LCD_CS
- R57 pad 2: /LCD_CS -> GND
- U1 pad 10: GND -> /power_in/PD_PG
- U1 pad 6: /power_in/CC2 -> /power_in/CC1
- U1 pad 7: /power_in/CC1 -> /power_in/CC2
- U17 pad 20: /LCD_CS -> /TAP_SEL_IO
- U17 pad 3: GND -> /mcu/ESP_EN
- U18 pad 1: GND -> /IR_IN
- U18 pad 3: /IR_IN -> /ui/IR_VCC
Routing:
- net GND: track 53.5 -> 298.5 mm, vias 261 -> 535
- net /linein/TAP_R: track 0.00 -> 58.1 mm, vias 0 -> 12
- net /A_SPK_L+: track 12.8 -> 65.3 mm
- net /A_SPK_R+: track 10.0 -> 47.6 mm
- net /LCD_CS: track 75.3 -> 38.1 mm, vias 2 -> 0
- net +5VA: track 85.6 -> 120.2 mm, vias 6 -> 10
- net /linein/ADC_SRC_L: track 0.00 -> 32.6 mm, vias 0 -> 6
- net /linein/ADC_SRC_R: track 0.00 -> 31.8 mm, vias 0 -> 7
- net /TAP_SEL_IO: track 0.00 -> 30.5 mm, vias 0 -> 2
- net /power_in/PD_PG: track 0.00 -> 26.7 mm, vias 0 -> 5
- net /VREF: track 26.5 -> 48.3 mm, vias 0 -> 4
- net /linein/TAP_L: track 0.00 -> 21.5 mm
- net /linein/ADC_LP: track 31.9 -> 10.9 mm
- net /mcu/ESP_EN: track 44.8 -> 63.3 mm, vias 2 -> 5
- net +3V3: track 69.3 -> 53.1 mm
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- added copper zone on F.Cu, net VBUS
- added copper zone on F.Cu, net VBUS_IN
